File: design_blocks/Power.kicad_blocks/Power Selection, 5V.kicad_block/Power Selection, 5V.kicad_sch (KiCad schematic)
At the start: 1 part, among them U2 LM66200DRLR

Commit message: Added additional parts; fixed origin of other parts
Added new design blocks
Parts:
- U2: FT Rotation Offset (none) -> -90
Changed lines of the file:
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@@
-			)
-		)
-		(property "Height" "0.6"
-			(at 51.308 96.012 0)
-			(effects
-				(font
-					(size 1.27 1.27)
-				)
-				(justify left top)
-				(hide yes)
 			)
 		)
@@
 			(effects
 				(font
+					(size 1.27 1.27)
+				)
+				(hide yes)
+			)
+		)
+		(property "Height" "0.6"
+			(at 51.308 96.012 0)
+			(effects
+				(font
+					(size 1.27 1.27)
+				)
+				(justify left top)
+				(hide yes)
+			)
+		)
+		(property "FT Rotation Offset" "-90"
+			(at 49.53 80.01 0)
+			(effects
+				(font
