File: design_blocks/Aquarius.kicad_blocks/Module MCU Block.kicad_block/Module MCU Block.kicad_sch (KiCad schematic)
At the start: 17 parts, among them U2 ATtiny1616-MNR

Commit message: Updated blocks
Added current sensor
Updated LEDs
Updated QWICC
Changed MCU
Parts:
- removed C3: .1uF, Capacitor_SMD:C_0603_1608Metric, symbol Device:C
- removed JP4: Jumper_3_Open, CRGM Connector:SolderJumper-3_P1.3mm_Open_RoundedPad1.0x1.5mm, symbol Jumper:Jumper_3_Open
- removed JP5: A0, CRGM Connector:SolderJumper-2_P1.3mm_Open_RoundedPad1.0x1.5mm, symbol Jumper:SolderJumper_2_Open
- removed JP6: A1, CRGM Connector:SolderJumper-2_P1.3mm_Open_RoundedPad1.0x1.5mm, symbol Jumper:SolderJumper_2_Open
- removed R8, R9: 4.7K, Resistor_SMD:R_0603_1608Metric, symbol Device:R_US
- removed TP17: PC2, CRGM Mechanical:TestPoint_Pad_D1.0mm, symbol Connector:TestPoint
- removed TP18: PC3, CRGM Mechanical:TestPoint_Pad_D1.0mm, symbol Connector:TestPoint
- removed TP19: PA1, CRGM Mechanical:TestPoint_Pad_D1.0mm, symbol Connector:TestPoint
- removed TP20: PA2, CRGM Mechanical:TestPoint_Pad_D1.0mm, symbol Connector:TestPoint
- removed TP21: PA3, CRGM Mechanical:TestPoint_Pad_D1.0mm, symbol Connector:TestPoint
- removed TP22: PA4, CRGM Mechanical:TestPoint_Pad_D1.0mm, symbol Connector:TestPoint
- removed TP23: PA5, CRGM Mechanical:TestPoint_Pad_D1.0mm, symbol Connector:TestPoint
- removed TP24: PA6, CRGM Mechanical:TestPoint_Pad_D1.0mm, symbol Connector:TestPoint
- removed TP25: PA7, CRGM Mechanical:TestPoint_Pad_D1.0mm, symbol Connector:TestPoint
- removed TP26: PC1, CRGM Mechanical:TestPoint_Pad_D1.0mm, symbol Connector:TestPoint
- removed U2: ATtiny1616-MNR, CRG Makes:VQFN-20-1EP_3x3mm_P0.4mm_EP1.7x1.7mm_ThermalVias, symbol CRG Makes:ATtiny1616-MNR
- added C1: .1uF, CRGM Passive:C_0603_1608Metric, symbol Device:C
- added JP1: ~, CRGM Connector:SolderJumper-3_P1.3mm_Open_RoundedPad1.0x1.5mm, symbol Jumper:Jumper_3_Open
- added JP2, JP3: ~, CRGM Connector:SolderJumper-2_P1.3mm_Open_RoundedPad1.0x1.5mm, symbol Jumper:SolderJumper_2_Open
- added R3, R4: 4.7K, CRGM Passive:R_0603_1608Metric, symbol Device:R_US
- added TP10, TP11, TP12, TP13, TP14, TP6, TP7, TP8, TP9: ~, CRGM Mechanical:TestPoint_Pad_D1.0mm, symbol CRGM Connector:TestPoint
- added U1: ATtiny1616-MNR, CRG Makes:VQFN-20-1EP_3x3mm_P0.4mm_EP1.7x1.7mm_ThermalVias, symbol CRG Makes:ATtiny1616-MNR
Connections:
- net +3.3V: now also C1.1, JP1.2 (C), U1.4 (VCC)
- net A0: now also JP2.2 (B), U1.10 (PB4/0OUT)
- net A1: now also JP3.2 (B), U1.9 (PB5/CLK0)
- net GND: now also C1.2, JP2.1 (A), JP3.1 (A), U1.21 (GND), U1.3 (GND)
- net PA1: now also TP8.1, U1.20 (MOSI/PA1)
- net PA2: now also TP9.1, U1.1 (MISO/PA2)
- net PA3: now also TP10.1, U1.2 (SCK/PA3)
- net PA4: now also TP11.1, U1.5 (~{SS}/PA4)
- net PA5: now also TP12.1, U1.6 (VREF/PA5)
- net PA6: now also TP13.1, U1.7 (DAC/PA6)
- net PA7: now also TP14.1, U1.8 (1OUT/PA7)
- net PC2: now also TP6.1, U1.17 (PC2)
- net PC3: now also TP7.1, U1.18 (PC3)
- net RXD: now also U1.11 (PB3/RxD)
- net SCL: now also R3.1, U1.14 (PB0/SCL)
- net SDA: now also R4.1, U1.13 (PB1/SDA)
- net TXD: now also U1.12 (PB2/TxD)
- net UPDI: now also U1.19 (UPDI/PA0)
- new net: JP1.1 (A), R3.2
- new net: JP1.3 (B), R4.2
- new net RELAY_EN: U1.16 (PC1)
- new net RELAY_LED: U1.15 (PC0/SCLK)
